Commit message: Added joints - Not tested

File: surgical_robot_description/urdf/surgical_robot.urdf (robot description, URDF)
Before this commit: robot surgical_robot, 11 links, 12 joints
Joints:
- joint joint1: origin xyz=-0.021 0.04806 0.01395 rpy=0 0 0 -> xyz=-0.021 0.01395 -0.04806  rpy=0 0 0
- joint joint10: origin xyz=0.0185 -0.00839 0.08 rpy=0 0 0 -> xyz=0.0185 0.08 0.00839 rpy=0 0 0
- joint joint11: origin xyz=0.16 0.01508 0.0185 rpy=0 0 0 -> xyz=0.16 0.0185 -0.01508 rpy=0 0 0
- joint joint12: origin xyz=0.16 0.00719 0 rpy=0 0 0 -> xyz=0.16 0 -0.00719 rpy=0 0 0
- joint joint2: axis (none) -> 1 0 0; limit (none) -> lower=0 upper=0.1 effort=0.001 velocity=0.2; origin xyz=0.006 0.055 0.00995 rpy=0 0 0 -> xyz=0.006  0.00995 -0.055 rpy=0 0 0; type fixed -> prismatic
- joint joint3: axis (none) -> 0 1 0; limit (none) -> lower=0 upper=0.1 effort=0.001 velocity=0.2; origin xyz=0.0343 0.0054 0.01195 rpy=0 0 0 -> xyz=0.0343 0.01195 -0.0054 rpy=0 0 0; type fixed -> prismatic
- joint joint4: axis  -> 0 0 1; limit (none) -> lower=0 upper=0.1 effort=0.001 velocity=0.2; origin xyz=0.011 -0.007 0.04381 rpy=0 0 0 -> xyz=0.011 0.04381 0.007 rpy=0 0 0; type fixed -> prismatic
- joint joint5: origin xyz=0.0492 0.131 0.07602 rpy=0 0 0 -> xyz=0.0492 0.07602 -0.131 rpy=0 0 0
- joint joint6: origin xyz=0.00724 -0.0821 0.02398 rpy=0 0 0 -> xyz=0.00724 0.02398 0.0821 rpy=0 0 0
- joint joint7: origin xyz=-0.01126 -0.0901 0.02398 rpy=0 0 0 -> xyz=-0.01126 0.02398 0.0901 rpy=0 0 0
- joint joint8: origin xyz=0 -0.01639 0.08 rpy=0 0 0 -> xyz=0 0.08 0.01639 rpy=0 0 0
- joint joint9: origin xyz=0 -0.0085 0.0985 rpy=0 0 0 -> xyz=0 0.0985 0.0085 rpy=0 0 0

Commit message: Modified joints to fix RCM

File: surgical_robot_description/urdf/surgical_robot.urdf (robot description, URDF)
Before this commit: robot surgical_robot, 11 links, 12 joints
Links:
- added link needle_eef; collision cylinder length=0.02 radius=0.0022; visual cylinder length=0.0025 radius=0.0022
- added link needle_link; collision cylinder length=0.12 radius=0.0022; visual cylinder length=0.12 radius=0.0022
- link axial_translation: mass None -> 0.5
- link base: mass None -> 0.5; geometry collision mesh filename=package://surgical_robot_description/meshes/base.stl; visual mesh filename=package://surgical_robot_description/meshes/base_200.stl
- link base_link: mass None -> 0.5; geometry collision mesh filename=package://surgical_robot_description/meshes/MRI_2000.stl; visual mesh filename=package://surgical_robot_description/meshes/MRI.stl
- link base_yaw: mass None -> 0.5; geometry collision mesh filename=package://surgical_robot_description/meshes/base_yaw.stl; visual mesh filename=package://surgical_robot_description/meshes/base_yaw_200.stl
- link horizontal_long: mass None -> 0.5
- link horizontal_short: mass None -> 0.5
- link lateral_translation: mass None -> 0.5
- link needle_driver: mass None -> 0.5; geometry visual mesh filename=package://surgical_robot_description/meshes/needle_driver_2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
- link vertical_long: mass None -> 0.5; geometry collision mesh filename=package://surgical_robot_description/meshes/vertical_long.s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; visual mesh filename=package://surgical_robot_description/meshes/vertical_long_2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
- link vertical_short: mass None -> 0.5; geometry collision mesh filename=package://surgical_robot_description/meshes/vertical_short.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; visual mesh filename=package://surgical_robot_description/meshes/vertical_short_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
- link vertical_translation: mass None -> 0.5
Joints:
- removed joint joint10
- added joint joint13: type revolute, parent needle_driver, child needle_link, origin xyz=0 -0.03 -0.03719 rpy=1.57 0 0, axis 0 1 0, limit lower=-0.5 upper=0.5 effort=1000.0 velocity=0.5, mimic joint=joint7 multiplier=1 offset=0
- added joint joint14: type fixed, parent needle_link, child needle_eef, origin xyz=0 0 0.06125 rpy=0 0 0
- joint joint11: axis (none) -> 0 1 0; limit (none) -> lower=0 upper=0.1 effort=0.001 velocity=0.2; type fixed -> prismatic
- joint joint12: axis (none) -> 0 1 0; limit (none) -> lower=0 upper=0.1 effort=0.001 velocity=0.2; type fixed -> prismatic
- joint joint2: axis 1 0 0 -> 0 0 1
- joint joint3: axis 0 1 0 -> 1 0 0
- joint joint4: axis 0 0 1 -> 0 1 0
- joint joint5: axis (none) -> 1 0 0; limit (none) -> lower=-0.5 upper=0.5 effort=1000.0 velocity=0.5; origin xyz=0.0492 0.07602 -0.131 rpy=0 0 0 -> xyz=0.0777 0.10202 -0.086 rpy=0 0 0; type fixed -> revolute
- joint joint6: axis (none) -> 0 0 1; limit (none) -> lower=-0.5 upper=0.5 effort=1000.0 velocity=0.5; mimic (none) -> joint=joint7 multiplier=1 offset=0; origin xyz=0.00724 0.02398 0.0821 rpy=0 0 0 -> xyz=-0.02126 -0.00202 0.0371 rpy=0 0 0; type fixed -> revolute
- joint joint7: axis (none) -> 0 0 1; limit (none) -> lower=-0.5 upper=0.5 effort=1000.0 velocity=0.5; origin xyz=-0.01126 0.02398 0.0901 rpy=0 0 0 -> xyz=-0.03976 -0.00202 0.0451 rpy=0 0 0; type fixed -> revolute
- joint joint8: axis (none) -> 0 0 1; limit (none) -> lower=-0.5 upper=0.5 effort=1000.0 velocity=0.5; mimic (none) -> joint=joint7 multiplier=-1 offset=0; type fixed -> revolute
- joint joint9: axis (none) -> 0 0 1; limit (none) -> lower=-0.5 upper=0.5 effort=1000.0 velocity=0.5; mimic (none) -> joint=joint7 multiplier=-1 offset=0; type fixed -> revolute

Commit message: Intermideate save to keep a backup of urdf file

File: surgical_robot_description/urdf/surgical_robot.urdf (robot description, URDF)
Before this commit: robot surgical_robot_description, 13 links, 13 joints
Joints:
- removed joint joint1
- removed joint joint11
- removed joint joint12
- removed joint joint13
- removed joint joint14
- removed joint joint2
- removed joint joint3
- removed joint joint4
- removed joint joint5
- removed joint joint6
- removed joint joint7
- removed joint joint8
- removed joint joint9
- added joint MRI_base_frame: type fixed, parent base_link, child axial_translation, origin xyz=-0.021 0.01395 -0.04806  rpy=0 0 0
- added joint base_vertical_long: type revolute, parent base_yaw, child vertical_long, origin xyz=-0.02126 -0.00202 0.0371 rpy=0 0 0, axis 0 0 1, limit lower=-0.5 upper=0.5 effort=1000.0 velocity=0.5, mimic joint=base_vertical_short multiplier=1 offset=0
- added joint base_vertical_short: type revolute, parent base_yaw, child vertical_short, origin xyz=-0.03976 -0.00202 0.0451 rpy=0 0 0, axis 0 0 1, limit lower=-0.5 upper=0.5 effort=1000.0 velocity=0.5
- added joint base_x: type prismatic, parent axial_translation, child lateral_translation, origin xyz=0.006  0.00995 -0.055 rpy=0 0 0, axis 0 0 1, limit lower=0 upper=0.1 effort=0.001 velocity=0.2
- added joint base_y: type prismatic, parent lateral_translation, child vertical_translation, origin xyz=0.0343 0.01195 -0.0054 rpy=0 0 0, axis 1 0 0, limit lower=0 upper=0.1 effort=0.001 velocity=0.2
- added joint base_yaw: type revolute, parent base, child base_yaw, origin xyz=0.0777 0.10202 -0.086 rpy=0 0 0, axis 1 0 0, limit lower=-0.5 upper=0.5 effort=1000.0 velocity=0.5
- added joint base_z: type prismatic, parent vertical_translation, child base, origin xyz=0.011 0.04381 0.007 rpy=0 0 0, axis 0 1 0, limit lower=0 upper=0.1 effort=0.001 velocity=0.2
- added joint horizontal_l_needle_d: type prismatic, parent horizontal_long, child needle_driver, origin xyz=0.16 0.0185 -0.01508 rpy=0 0 0, axis 0 1 0, limit lower=0 upper=0.1 effort=0.001 velocity=0.2
- added joint horizontal_l_vertical_s: type revolute, parent vertical_short, child horizontal_long, origin xyz=0.0185 0.08 0.00839 rpy=0 0 0, axis 0 0 1, limit lower=-0.5 upper=0.5 effort=1000.0 velocity=0.5
- added joint horizontal_s_needle_d: type prismatic, parent horizontal_short, child needle_driver, origin xyz=0.16 0 -0.00719 rpy=0 0 0, axis 0 1 0, limit lower=0 upper=0.1 effort=0.001 velocity=0.2
- added joint horizontal_s_vertical_l: type revolute, parent vertical_long, child horizontal_short, origin xyz=0 0.0985 0.0085 rpy=0 0 0, axis 0 0 1, limit lower=-0.5 upper=0.5 effort=1000.0 velocity=0.5, mimic joint=base_vertical_short multiplier=-1 offset=0
- added joint horizontal_vertical_long: type revolute, parent vertical_long, child horizontal_long, origin xyz=0 0.08 0.01639 rpy=0 0 0, axis 0 0 1, limit lower=-0.5 upper=0.5 effort=1000.0 velocity=0.5, mimic joint=base_vertical_short multiplier=-1 offset=0
- added joint needle_d_needle_l: type revolute, parent needle_driver, child needle_link, origin xyz=0 -0.03 -0.03719 rpy=1.57 0 0, axis 0 1 0, limit lower=-0.5 upper=0.5 effort=1000.0 velocity=0.5, mimic joint=base_vertical_short multiplier=1 offset=0
- added joint needle_l_needle_e: type fixed, parent needle_link, child needle_eef, origin xyz=0 0 0.06125 rpy=0 0 0

Commit message: Added world frame to fix the spawn state

File: surgical_robot_description/urdf/surgical_robot.urdf (robot description, URDF)
Before this commit: robot surgical_robot_description, 13 links, 14 joints
Links:
- added link world
Joints:
- added joint world_link: type fixed, parent world, child base_link, origin xyz=0 0 0 rpy=1.5707 0 3.14, axis 0 -0.5 0

Commit message: Update surgical_robot.urdf
Corrected joint positions for:
base_yaw
base_vertical_long
base_vertical_short

Swapped "visual" and "collision" geometry links so that higher fidelity models are used for visual and lower fidelity models are used for collisions.

Adjusted joint lower and upper limits to be more realistic

File: surgical_robot_description/urdf/surgical_robot.urdf (robot description, URDF)
Before this commit: robot surgical_robot_description, 14 links, 15 joints
Links:
- link base: geometry collision mesh filename=package://surgical_robot_description/meshes/base_200.stl; visual mesh filename=package://surgical_robot_description/meshes/base.stl
- link base_link: geometry collision mesh filename=package://surgical_robot_description/meshes/MRI.stl; visual mesh filename=package://surgical_robot_description/meshes/MRI_2000.stl
- link base_yaw: geometry collision mesh filename=package://surgical_robot_description/meshes/base_yaw_200.stl; visual mesh filename=package://surgical_robot_description/meshes/base_yaw.stl
- link needle_driver: geometry visual mesh filename=package://surgical_robot_description/meshes/needle_driver.s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
- link vertical_long: geometry collision mesh filename=package://surgical_robot_description/meshes/vertical_long_2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; visual mesh filename=package://surgical_robot_description/meshes/vertical_long.s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
- link vertical_short: geometry collision mesh filename=package://surgical_robot_description/meshes/vertical_short_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; visual mesh filename=package://surgical_robot_description/meshes/vertical_short.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
Joints:
- joint base_vertical_long: limit lower=-0.5 upper=0.5 effort=1000.0 velocity=0.5 -> lower=-0.52 upper=0.52 effort=1000.0 velocity=0.5; origin xyz=-0.02126 -0.00202 0.0371 rpy=0 0 0 -> xyz=-0.01925 0.000 0.02781 rpy=0 0 0
- joint base_vertical_short: limit lower=-0.5 upper=0.5 effort=1000.0 velocity=0.5 -> lower=-0.52 upper=0.52 effort=1000.0 velocity=0.5; origin xyz=-0.03976 -0.00202 0.0451 rpy=0 0 0 -> xyz=-0.03775 0.000 0.03581 rpy=0 0 0
- joint base_x: limit lower=0 upper=0.1 effort=0.001 velocity=0.2 -> lower=0 upper=0.05 effort=0.001 velocity=0.2
- joint base_y: limit lower=0 upper=0.1 effort=0.001 velocity=0.2 -> lower=-0.02 upper=0.02 effort=0.001 velocity=0.2
- joint base_yaw: limit lower=-0.5 upper=0.5 effort=1000.0 velocity=0.5 -> lower=-0.52 upper=0.52 effort=1000.0 velocity=0.5; origin xyz=0.0777 0.10202 -0.086 rpy=0 0 0 -> xyz=0.07569 0.100 -0.078 rpy=0 0 0
- joint base_z: limit lower=0 upper=0.1 effort=0.001 velocity=0.2 -> lower=-0.02 upper=0.05 effort=0.001 velocity=0.2
- joint horizontal_l_needle_d: limit lower=0 upper=0.1 effort=0.001 velocity=0.2 -> lower=-0.05 upper=0.05 effort=0.001 velocity=0.2
- joint horizontal_l_vertical_s: limit lower=-0.5 upper=0.5 effort=1000.0 velocity=0.5 -> lower=-0.52 upper=0.52 effort=1000.0 velocity=0.5
- joint horizontal_s_needle_d: limit lower=0 upper=0.1 effort=0.001 velocity=0.2 -> lower=-0.05 upper=0.05 effort=0.001 velocity=0.2
- joint horizontal_s_vertical_l: limit lower=-0.5 upper=0.5 effort=1000.0 velocity=0.5 -> lower=-0.52 upper=0.52 effort=1000.0 velocity=0.5
- joint horizontal_vertical_long: limit lower=-0.5 upper=0.5 effort=1000.0 velocity=0.5 -> lower=-0.52 upper=0.52 effort=1000.0 velocity=0.5
- joint needle_d_needle_l: limit lower=-0.5 upper=0.5 effort=1000.0 velocity=0.5 -> lower=-0.52 upper=0.52 effort=1000.0 velocity=0.5

Commit message: Configured moveit with the URDF file and fixed the URDF file

File: surgical_robot_description/urdf/surgical_robot.urdf (robot description, URDF)
Before this commit: robot surgical_robot_description, 14 links, 15 joints
Joints:
- removed joint base_vertical_short
- removed joint horizontal_l_needle_d
- removed joint horizontal_l_vertical_s
- added joint base_pitch: type revolute, parent base_yaw, child vertical_short, origin xyz=-0.03775 0.000 0.03581 rpy=0 0 0, axis 0 0 1, limit lower=-0.52 upper=0.52 effort=1000.0 velocity=0.5
- joint base_vertical_long: mimic joint=base_vertical_short multiplier=1 offset=0 -> joint=base_pitch multiplier=1 offset=0
- joint horizontal_s_needle_d: axis 0 1 0 -> 0 0 1; mimic (none) -> joint=base_pitch multiplier=1 offset=0; type prismatic -> revolute
- joint horizontal_s_vertical_l: mimic joint=base_vertical_short multiplier=-1 offset=0 -> joint=base_pitch multiplier=-1 offset=0
- joint horizontal_vertical_long: mimic joint=base_vertical_short multiplier=-1 offset=0 -> joint=base_pitch multiplier=-1 offset=0
- joint needle_d_needle_l: axis 0 1 0 -> (none); limit lower=-0.52 upper=0.52 effort=1000.0 velocity=0.5 -> (none); mimic joint=base_vertical_short multiplier=1 offset=0 -> (none); type revolute -> fixed
